Commit message: add sdf

File: ouster_os1_64/urdf/os1_64.urdf.xacro (robot description, xacro)
@@ -38,5 +38,5 @@
         <origin xyz="0 0 0" rpy="0 0 0"/>
         <geometry>
-          <mesh filename="package://ouster_os1_64/meshes/${file_visual}.stl" />
+          <mesh filename="package://ouster_os1_64/models/os1_32/meshes/${file_visual}.stl" />
         </geometry>
       </visual>
